File: Hackpad.kicad_pcb (KiCad board)
At the start: 2 copper layers, 146.8 x 116.7 mm, 51 parts, among them Q1 SW_Push, U1 MOUDLE-SEEEDUINO-XIAO

Commit message: 3d model and firmware compiled
Parts:
- removed ?: LOGO, Hackpad:pfp
Connections:
- U1 pad 10: ROW3 -> ROW2
- U1 pad 11: ROW2 -> ROW1
- U1 pad 12: ROW1 -> unconnected-(U1-3V3-Pad12)
- U1 pad 6: unconnected-(U1-PA9_A5_D5_SCL-Pad6) -> LED
- U1 pad 8: LED -> ROW4
- U1 pad 9: ROW4 -> ROW3
Routing:
- net +5V: track 407.2 -> 474.5 mm, vias 13 -> 15
- net LED: track 14.6 -> 49.8 mm
- net ROW4: track 80.9 -> 79.0 mm
- net ROW3: track 77.8 -> 76.2 mm
- net ROW2: track 61.4 -> 60.3 mm
- net ROW1: track 45.7 -> 44.7 mm
- net Net-(D6-A): track 117.0 -> 117.9 mm
- net Net-(D7-A): track 85.3 -> 86.2 mm
- net GND: vias 0 -> 300
- added copper zone on B.Cu, net GND
Other:
- outline, holes or cut-outs redrawn
